File: KITKADADC.kicad_sch (KiCad schematic)
At the start: 0 parts

Commit message: he puesto un diodo
Parts:
- added D1, D2: 1N47xxA, Diode_THT:D_DO-41_SOD81_P10.16mm_Horizontal, symbol Diode:1N47xxA
Changed lines of the file:
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@@
 	(generator_version "10.0")
 	(paper "A4")
+	(symbol
+		(lib_id "Diode:1N47xxA")
+		(at -15.24 36.83 0)
+		(unit 1)
+		(body_style 1)
+		(exclude_from_sim no)
+		(in_bom yes)
+		(on_board yes)
+		(in_pos_files yes)
+		(dnp no)
+		(fields_autoplaced yes)
+		(property "Reference" "D1"
+			(at -15.24 30.48 0)
+			(show_name no)
+			(do_not_autoplace no)
+			(effects
+				(font
+					(size 1.27 1.27)
+				)
+			)
+		)
+		(property "Value" "1N47xxA"
+			(at -15.24 33.02 0)
+			(show_name no)
+			(do_not_autoplace no)
+			(effects
+				(font
+					(size 1.27 1.27)
+				)
+			)
+		)
+		(property "Footprint" "Diode_THT:D_DO-41_SOD81_P10.16mm_Horizontal"
+			(at -15.24 41.275 0)
+			(hide yes)
+			(show_name no)
+			(do_not_autoplace no)
+			(effects
+				(font
+					(size 1.27 1.27)
+				)
+			)
+		)
+		(property "Datasheet" "https://www.vishay.com/docs/85816/1n4728a.pdf"
+			(at -15.24 36.83 0)
+			(hide yes)
+			(show_name no)
+			(do_not_autoplace no)
+			(effects
+				(font
+					(size 1.27 1.27)
+				)
+			)
+		)
+		(property "Description" "1300mW Silicon planar power Zener diodes, DO-41"
+			(at -15.24 36.83 0)
+			(hide yes)
+			(show_name no)
+			(do_not_autoplace no)
+			(effects
+				(font
+					(size 1.27 1.27)
+				)
+			)
+		)
+		(pin "1"
+		)
+		(pin "2"
+		)
+		(instances
+			(project "KITKADADC"
+				(path "/7abc5919-1e50-493f-9841-d705b6442d51"
+					(reference "D1")
+					(unit 1)
+				)
+			)
+		)
+	)
+	(symbol
+		(lib_id "Diode:1N47xxA")
+		(at 109.22 72.39 0)
+		(unit 1)
+		(body_style 1)
+		(exclude_from_sim no)
+		(in_bom yes)
+		(on_board yes)
+		(in_pos_files yes)
+		(dnp no)
+		(fields_autoplaced yes)
+		(property "Reference" "D2"
+			(at 109.22 66.04 0)
+			(show_name no)
+			(do_not_autoplace no)
+			(effects
+				(font
+					(size 1.27 1.27)
+				)
+			)
+		)
+		(property "Value" "1N47xxA"
+			(at 109.22 68.58 0)
+			(show_name no)
+			(do_not_autoplace no)
+			(effects
+				(font
+					(size 1.27 1.27)
+				)
+			)
+		)
+		(property "Footprint" "Diode_THT:D_DO-41_SOD81_P10.16mm_Horizontal"
+			(at 109.22 76.835 0)
+			(hide yes)
+			(show_name no)
+			(do_not_autoplace no)
+			(effects
+				(font
+					(size 1.27 1.27)
+				)
+			)
+		)
+		(property "Datasheet" "https://www.vishay.com/docs/85816/1n4728a.pdf"
+			(at 109.22 72.39 0)
+			(hide yes)
+			(show_name no)
+			(do_not_autoplace no)
+			(effects
+				(font
+					(size 1.27 1.27)
+				)
+			)
+		)
+		(property "Description" "1300mW Silicon planar power Zener diodes, DO-41"
+			(at 109.22 72.39 0)
+			(hide yes)
+			(show_name no)
+			(do_not_autoplace no)
+			(effects
+				(font
+					(size 1.27 1.27)
+				)
+			)
+		)
+		(pin "2"
+		)
+		(pin "1"
+		)
+		(instances
+			(project "KITKADADC"
+				(path "/7abc5919-1e50-493f-9841-d705b6442d51"
+					(reference "D2")
+					(unit 1)
+				)
+			)
+		)
+	)
 	(sheet_instances
 		(path "/"

Commit message: empezando con el adc
Parts:
- removed D1, D2: 1N47xxA, Diode_THT:D_DO-41_SOD81_P10.16mm_Horizontal, symbol Diode:1N47xxA
- added C1, C10, C11, C12, C16, C17, C18, C19, C2, C3, C4, C5, C6, C7, C8, C9: 100nF, Capacitor_SMD:C_0402_1005Metric, symbol Device:C
- added C13, C14, C15, C20: 10nF, Capacitor_SMD:C_0603_1608Metric, symbol Device:C
- added D1, D2, D3, D5: SRV05-4, Package_TO_SOT_SMD:SOT-23-6, symbol Power_Protection:NUP4202
- added D4: LED-RED, LED_SMD:LED_0603_1608Metric, symbol Device:LED
- added FID1, FID2: Fiducial, Fiducial:Fiducial_0.5mm_Mask1mm, symbol Mechanical:Fiducial
- added R1, R38, R40: DNP, Resistor_SMD:R_0402_1005Metric, symbol Device:R
- added R10, R12, R13, R7: 2.7k, Resistor_SMD:R_0603_1608Metric, symbol Device:R
- added R11, R2, R3, R39, R4, R42, R5, R6, R8, R9: 470K, Resistor_SMD:R_0402_1005Metric, symbol Device:R
- added R14, R15, R16, R17, R18, R19, R20, R21, R22, R23, R24, R25, R45, R46, R47, R48: 6.8K, Resistor_SMD:R_0603_1608Metric, symbol Device:R
- added R26, R27, R28, R29, R30, R31, R32, R33, R34, R35, R36, R37, R43, R49, R50, R51, R52: 10K, Resistor_SMD:R_0603_1608Metric, symbol Device:R
- added R41: 2.2k, Resistor_SMD:R_0603_1608Metric, symbol Device:R
- added R44: 39k, Resistor_SMD:R_0603_1608Metric, symbol Device:R
- added RN1, RN2, RN3, RN4: 10k, Resistor_SMD:R_Array_Convex_4x0603, symbol Device:R_Pack04
- added U1, U10, U11, U12, U13, U14, U15, U16, U17, U18, U19, U2, U20, U3, U4, U5, U6, U7, U8, U9: MCP6004, Package_SO:TSSOP-14_4.4x5mm_P0.65mm, symbol Amplifier_Operational:MCP6004
Connections:
- new net: R20.2, U8.1, U8.2 (-)
- new net: C9.1, D3.3, RN2.6 (R3.2), U8.3 (+)
- new net: R21.2, U9.1, U9.2 (-)
- new net: C11.1, D3.1, RN2.5 (R4.2), U9.3 (+)
- new net: R18.2, U6.1, U6.2 (-)
- new net: C5.1, D3.6, RN2.8 (R1.2), U6.3 (+)
- new net: R19.2, U7.1, U7.2 (-)
- new net: C7.1, D3.4, RN2.7 (R2.2), U7.3 (+)
- new net: R16.2, U3.1, U3.2 (-)
- new net: C3.1, D1.3, RN1.6 (R3.2), U3.3 (+)
- new net: R17.2, U4.1, U4.2 (-)
- new net: C4.1, D1.1, RN1.5 (R4.2), U4.3 (+)
- new net: R14.2, U1.1, U1.2 (-)
- new net: C1.1, D1.6, RN1.8 (R1.2), U1.3 (+)
- new net: R15.2, U2.1, U2.2 (-)
- new net: C2.1, D1.4, RN1.7 (R2.2), U2.3 (+)
- new net: R22.2, U10.1, U10.2 (-)
- new net: C6.1, D2.3, RN3.8 (R1.2), U10.3 (+)
- new net: R23.2, U11.1, U11.2 (-)
- new net: C8.1, D2.1, RN3.7 (R2.2), U11.3 (+)
- new net: R24.2, U12.1, U12.2 (-)
- new net: C10.1, D2.6, RN3.6 (R3.2), U12.3 (+)
- new net: R25.2, U13.1, U13.2 (-)
- new net: C12.1, D2.4, RN3.5 (R4.2), U13.3 (+)
- new net: D4.1 (K), R41.2
- new net: R45.2, U16.1, U16.2 (-)
- new net: C16.1, D5.3, RN4.8 (R1.2), U16.3 (+)
- new net: R46.2, U17.1, U17.2 (-)
- new net: C17.1, D5.1, RN4.7 (R2.2), U17.3 (+)
- new net: R47.2, U18.1, U18.2 (-)
- new net: C18.1, D5.6, RN4.6 (R3.2), U18.3 (+)
- new net: R48.2, U19.1, U19.2 (-)
- new net: R43.1, R44.1, RN4.3 (R3.1)
- new net 12V: R44.2
- new net 5V: C13.1, C14.1, C15.1, C20.1, D1.5, D2.5, D3.5, D4.2 (A), D5.5, R1.1, R10.2, R12.2, R13.2, R38.2, R40.2, R7.2
- new net AGND: R26.1, R27.1, R28.1, R29.1, R30.1, R31.1, R32.1, R33.1, R34.1, R35.1, R36.1, R37.1, R49.1, R50.1, R51.1, R52.1
- new net AT1: R13.1, RN2.4 (R4.1)
- new net AT1_MCU: R21.1, R37.2
- new net AT2: R12.1, RN2.3 (R3.1)
- new net AT2_MCU: R20.1, R36.2
- new net AT3: R10.1, RN2.2 (R2.1)
- new net AT3_MCU: R19.1, R35.2
- new net AT4: R7.1, RN2.1 (R1.1)
- new net AT4_MCU: R18.1, R34.2
- new net AV1: R11.1, RN3.4 (R4.1)
- new net AV10: R8.1, RN3.3 (R3.1)
- new net AV10_MCU: R24.1, R32.2
- new net AV11_MCU: R48.1, R52.2
- new net AV1_MCU: R25.1, R33.2
- new net AV2: R5.1, RN3.2 (R2.1)
- new net AV2_MCU: R23.1, R31.2
- new net AV3: R3.1, RN3.1 (R1.1)
- new net AV3_MCU: R22.1, R30.2
- new net AV4: R38.1, R39.1, RN4.2 (R2.1)
- new net AV4_MCU: R46.1, R50.2
- new net AV5: R40.1, R42.1, RN4.1 (R1.1)
- new net AV5_MCU: R45.1, R49.2
- new net AV6: R9.1, RN1.4 (R4.1)
- new net AV6_MCU: R17.1, R29.2
- new net AV7: R6.1, RN1.3 (R3.1)
- new net AV7_MCU: R16.1, R28.2
- new net AV8: R4.1, RN1.2 (R2.1)
- new net AV8_MCU: R15.1, R27.2
- new net AV9: R1.2, R2.1, RN1.1 (R1.1)
- new net AV9_MCU: R14.1, R26.2
- new net CAM: R41.1, RN4.4 (R4.1)
- new net CAM_MCU: C19.1, D5.4, RN4.5 (R4.2), U19.3 (+)
- new net GND: C1.2, C10.2, C11.2, C12.2, C13.2, C14.2, C15.2, C16.2, C17.2, C18.2, C19.2, C2.2, C20.2, C3.2, C4.2, C5.2, C6.2, C7.2, C8.2, C9.2, D1.2, D2.2, D3.2, D5.2, R11.2, R2.2, R3.2, R39.2, R4.2, R42.2, R43.2, R5.2, R6.2, R8.2, R9.2
- new net Vbat_MCU: R47.1, R51.2
Other:
- note added: "Comparator with histeresis for CAM input? Usign this OpAmp."
- note added: "NOT OEM POPULATED OEM IS AV6 AND AV10 ARE ANALOG AV8 AND AV9 ARE DIGITAL OUTPUTS"
- company: (none) -> rusEFI.com
- title: (none) -> microRusEFI-2L

Commit message: recolocando pcb
Parts:
- renumbered C1 to C16, C14 to C40, C2 to C45, C3 to C46, C4 to C47, C6 to C48, C8 to C49, C10 to C50, C12 to C51, C5 to C52, C7 to C53, C9 to C54, C11 to C55, C16 to C56, C17 to C57, C18 to C58, C19 to C59, C15 to C79, C13 to C80, C20 to C82, D1 to D13, D4 to D29, D3 to D38, D2 to D39, D5 to D40, FID1 to FID5, FID2 to FID6, R38 to R11, R39 to R131, R44 to R139, R7 to R14, R43 to R141, R10 to R23, R3 to R24, R12 to R25, R23 to R26, R13 to R27, R41 to R28, R5 to R31, R24 to R32, R8 to R34, R25 to R35, R11 to R37, R30 to R38, R31 to R39, R42 to R41, R32 to R44, R33 to R46, R22 to R5, R2 to R52, R14 to R53, R4 to R54, R15 to R55, R6 to R56, R16 to R57, R9 to R58, R17 to R59, R26 to R60, R27 to R61, R28 to R62, R29 to R63, R18 to R64, R19 to R65, R20 to R66, R21 to R67, R34 to R68, R35 to R69, R1 to R7, R36 to R70, R37 to R71, R45 to R72, R46 to R73, R47 to R74, R48 to R75, R49 to R76, R50 to R77, R51 to R78, R52 to R79, RN4 to RN13, RN1 to RN2, RN2 to RN3, RN3 to RN4, U8 to U35, U9 to U35, U6 to U35, U7 to U35, U15 to U35, U10 to U36, U11 to U36, U12 to U36, U13 to U36, U5 to U36, U16 to U46, U17 to U46, U18 to U46, U19 to U46, U20 to U46, U3 to U8, U4 to U8, U1 to U8, U2 to U8, U14 to U8
Connections:
- net 5V: now also U35.4 (V+), U36.4 (V+), U46.4 (V+), U8.4 (V+)
- net GND: now also U35.11 (V-), U36.11 (V-), U46.11 (V-), U8.11 (V-)
- net at C54.1, D38.3, RN3.6 (R3.2): now also U35.12 (+); no longer U35.3 (+)
- net at C55.1, D38.1, RN3.5 (R4.2): now also U35.10 (+); no longer U35.3 (+)
- net at C52.1, D38.6, RN3.8 (R1.2): now also U35.5 (+); no longer U35.3 (+)
- net at C46.1, D13.3, RN2.6 (R3.2): now also U8.12 (+); no longer U8.3 (+)
- net at C47.1, D13.1, RN2.5 (R4.2): now also U8.10 (+); no longer U8.3 (+)
- net at C16.1, D13.6, RN2.8 (R1.2): now also U8.5 (+); no longer U8.3 (+)
- net at C48.1, D39.3, RN4.8 (R1.2): now also U36.12 (+); no longer U36.3 (+)
- net at C49.1, D39.1, RN4.7 (R2.2): now also U36.10 (+); no longer U36.3 (+)
- net at C50.1, D39.6, RN4.6 (R3.2): now also U36.5 (+); no longer U36.3 (+)
- net at C56.1, D40.3, RN13.8 (R1.2): now also U46.12 (+); no longer U46.3 (+)
- net at C57.1, D40.1, RN13.7 (R2.2): now also U46.10 (+); no longer U46.3 (+)
- net at C58.1, D40.6, RN13.6 (R3.2): now also U46.5 (+); no longer U46.3 (+)
- new net: R66.2, U35.13 (-), U35.14
- new net: R67.2, U35.8, U35.9 (-)
- new net: R64.2, U35.6 (-), U35.7
- new net: R57.2, U8.13 (-), U8.14
- new net: R59.2, U8.8, U8.9 (-)
- new net: R53.2, U8.6 (-), U8.7
- new net: R5.2, U36.13 (-), U36.14
- new net: R26.2, U36.8, U36.9 (-)
- new net: R32.2, U36.6 (-), U36.7
- new net: R72.2, U46.13 (-), U46.14
- new net: R73.2, U46.8, U46.9 (-)
- new net: R74.2, U46.6 (-), U46.7
